File: PlantController/PlantController.sch (EAGLE design)
At the start: 42 parts, among them CON3 IMO_20.155MV/3, CON4 IMO_20.155MV/3, K3 RT314005, K4 RT314005, Q3 BS170, Q4 BS170

Commit message: * Made schematic consistent with BOM again.
Schematic part numbers got mixed up after simplifying the schemetic
resulting in an inconsistency with the BOM.
Parts:
- renumbered D1 to D3, D4 to D2, K3 to K1, K4 to K2, Q3 to Q1, Q4 to Q2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
Connections:
- net N$24 renamed K2
